File: STM32/STM32.kicad_pcb (KiCad board)
At the start: 2 copper layers, 1 part, among them U1 STM32F091RCTx

Commit message: Add files via upload
Parts:
- added Board1: Conn_02x06_Odd_Even, Connector_PinHeader_1.00mm:PinHeader_2x06_P1.00mm_Vertical, F.Cu at (145.8, 47.4)
- added Board2: Conn_02x06_Odd_Even, Connector_PinHeader_1.00mm:PinHeader_2x06_P1.00mm_Vertical, F.Cu at (150.2, 47.4)
- added Board3: Conn_02x06_Odd_Even, Connector_PinHeader_1.00mm:PinHeader_2x06_P1.00mm_Vertical, F.Cu at (154.5, 47.4)
- added Button1: ~, Button_Switch_SMD:SW_SPST_TL3342, F.Cu at (136.9, 62.0)
- added C1: 0.1uF, Capacitor_SMD:C_0603_1608Metric, F.Cu at (137.7, 81.0)
- added C10: 4.7uF, Capacitor_SMD:C_0603_1608Metric, F.Cu at (138.2, 57.2)
- added C2: 100nF, Capacitor_SMD:C_0603_1608Metric, F.Cu at (134.1, 49.6)
- added C3: 100nF, Capacitor_SMD:C_0603_1608Metric, F.Cu at (134.1, 52.1)
- added C4: 100nF, Capacitor_SMD:C_0603_1608Metric, F.Cu at (134.1, 54.7)
- added C5: 4.7uF, Capacitor_SMD:C_0603_1608Metric, F.Cu at (134.1, 57.2)
- added C6: 1uF, Capacitor_SMD:C_0603_1608Metric, F.Cu at (138.2, 47.1)
- added C7: C, Capacitor_SMD:C_0603_1608Metric, F.Cu at (138.2, 49.6)
- added C8: 10nF, Capacitor_SMD:C_0603_1608Metric, F.Cu at (138.2, 52.1)
- added C9: 100nF, Capacitor_SMD:C_0603_1608Metric, F.Cu at (138.2, 54.7)
- added Display(ILI9341TFT)1: Conn_01x08_Pin, Connector_PinHeader_1.00mm:PinHeader_1x08_P1.00mm_Vertical, F.Cu at (145.8, 55.5)
- added FB1: 600Ohm @ 100MHz, Resistor_SMD:R_0603_1608Metric, F.Cu at (142.2, 47.1)
- added J1: Conn_01x06_Pin, Connector_PinHeader_1.00mm:PinHeader_1x06_P1.00mm_Vertical, F.Cu at (145.8, 65.5)
- added J2: Conn_01x06_Pin, Connector_PinHeader_1.00mm:PinHeader_1x06_P1.00mm_Vertical, F.Cu at (149.2, 65.5)
- added J3: Conn_01x08_Pin, Connector_PinHeader_1.00mm:PinHeader_1x08_P1.00mm_Vertical, F.Cu at (149.2, 55.5)
- added J4: Conn_01x08_Pin, Connector_PinHeader_1.00mm:PinHeader_1x08_P1.00mm_Vertical, F.Cu at (152.5, 55.5)
- added Joystick1: Conn_01x05_Pin, Connector_PinHeader_1.00mm:PinHeader_1x05_P1.00mm_Vertical, F.Cu at (155.8, 55.5)
- added R1: 100k, Resistor_SMD:R_0603_1608Metric, F.Cu at (142.2, 49.6)
- added R2: 100k, Resistor_SMD:R_0603_1608Metric, F.Cu at (142.2, 52.1)
- added R3: R_US, Resistor_SMD:R_0603_1608Metric, F.Cu at (142.2, 54.7)
- added STLink1: Conn_02x05_Odd_Even, Connector_PinHeader_1.00mm:PinHeader_2x05_P1.00mm_Vertical, F.Cu at (152.5, 65.5)
- added SW1: SW_Push, Button_Switch_SMD:SW_SPST_TL3342, F.Cu at (128.3, 79.9)
Connections:
- net /PB10 renamed /RST_3
- net /PB11 renamed /FAULT_3
- net /PB12 renamed /STEP_4
- net /PB13 renamed /DIR_4
- net /PB14 renamed /RST_4
- net /PB15 renamed /FAULT_4
- net /PB8 renamed /STEP_3
- net /PB9 renamed /DIR_3
- net /PC10 renamed /STEP_2
- net /PC11 renamed /DIR_2
- net /PC12 renamed /RST_2
- net /PC13 renamed /FAULT_2
- net /PC6 renamed /STEP_1
- net /PC7 renamed /DIR_1
- net /PC8 renamed /RST_1
- net /PC9 renamed /FAULT_1
- U1 pad 10: /PC2 -> /DC/RS
- U1 pad 11: /PC3 -> /SDI/MOSI
- U1 pad 13: /3VA -> VDDA
- U1 pad 14: /PA0 -> /OUT_1_1
- U1 pad 15: /PA1 -> /OUT_2_1
- U1 pad 16: /PA2 -> /OUT_3_1
- U1 pad 17: /PA3 -> /OUT_1_2
- U1 pad 20: /PA4 -> /OUT_2_2
- U1 pad 21: /PA5 -> /OUT_3_2
- U1 pad 22: /PA6 -> /OUT_1_3
- U1 pad 23: /PA7 -> /OUT_2_3
- U1 pad 24: /PC4 -> /SCK
- U1 pad 25: /PC5 -> /LED_T
- U1 pad 26: /PB0 -> /Button
- U1 pad 27: /PB1 -> /Y-pos
- U1 pad 28: /PB2 -> /X-pos
- U1 pad 3: /PC14 -> unconnected-(U1-PC14-Pad3)
- U1 pad 4: /PC15 -> unconnected-(U1-PC15-Pad4)
- U1 pad 41: /PA8 -> /OUT_3_3
- U1 pad 42: /PA9 -> /S0
- U1 pad 43: /PA10 -> /S1
- U1 pad 44: /PA11 -> /S2
- U1 pad 45: /PA12 -> /S3
- U1 pad 46: /PA13 -> /OE
- U1 pad 49: /PA14 -> /LED
- U1 pad 50: /PA15 -> /But
- U1 pad 55: /PB3 -> unconnected-(U1-PB3-Pad55)
- U1 pad 56: /PB4 -> unconnected-(U1-PB4-Pad56)
- U1 pad 57: /PB5 -> unconnected-(U1-PB5-Pad57)
- U1 pad 58: /PB6 -> unconnected-(U1-PB6-Pad58)
- U1 pad 59: /PB7 -> unconnected-(U1-PB7-Pad59)
- U1 pad 60: /BOOT0 PF11 -> /BOOT0
- U1 pad 8: /PC0 -> /CS
- U1 pad 9: /PC1 -> /RESET
